Commit message: cluster

File: genesis/assets/urdf/mydrone/bix3_new.urdf (robot description, URDF)
Before this commit: robot drone, 16 links, 15 joints
Links:
- link elevator_wing: geometry collision box name=elevator_wing_collision_0_box_0 size=0.010157782429633631 0.04067820937821903 0.45189990568774874; visual mesh filename=package://meshes/fixed_wing_elevator.stl name=elevator_wing_visual_0_shape_0 scale=0.001 0.001 0.001
- link fuselage: geometry collision box name=fuselage_collision_0_box_0 size=0.1828019342982094 0.9308553327391513 1.1216608317366152; visual mesh filename=package://meshes/fixed_wing_fuselage.stl name=fuselage_visual_0_shape_0 scale=0.001 0.001 0.001
- link fuselage_left_aileron_0: mass 0.018 -> 0.0
- link fuselage_right_aileron_0: mass 0.018 -> 0.0
- link left_aileron_wing: geometry collision box name=left_aileron_wing_collision_0_box_0 size=0.008591109754893968 0.045759573470045924 0.294065274911455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; visual mesh filename=package://meshes/fixed_wing_left_aileron.stl name=left_aileron_wing_visual_0_shape_0 scale=0.001 0.001 0.001
- link prop_frame_fuselage: geometry collision box name=prop_frame_fuselage_collision_0_box_0 size=0.017413210987132194 0.01960053634643555 0.1774701226438359; visual mesh filename=package://meshes/propeller.stl name=prop_frame_fuselage_visual_0_shape_0 scale=0.001 0.001 0.001
- link right_aileron_wing: geometry collision box name=right_aileron_wing_collision_0_box_0 size=0.008658796238186621 0.045776045380552494 0.298108503088926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; visual mesh filename=package://meshes/fixed_wing_right_aileron.stl name=right_aileron_wing_visual_0_shape_0 scale=0.001 0.001 0.001
- link rudder_wing: geometry collision box name=rudder_wing_collision_0_box_0 size=0.005011972583816545 0.02725749058997695 0.1553331759530388; visual mesh filename=package://meshes/fixed_wing_rudder.stl name=rudder_wing_visual_0_shape_0 scale=0.001 0.001 0.001
Joints:
- joint fixed_joint_prop_frame_fuselage: origin xyz=-0.458 0 -0.076 rpy=0 -0.105 3.14159 -> xyz=-0.458 0 -0.076 rpy=0 -0.1745329 3.14159
- joint joint_0__elevator_wing: limit lower=-0.3491 upper=0.3491 effort=20.0 velocity=5.4 -> lower=-0.3491 upper=0.3491 effort=0.26 velocity=5.4
- joint joint_0__rudder_wing: limit lower=-0.3491 upper=0.3491 effort=20.0 velocity=5.4 -> lower=-0.3491 upper=0.3491 effort=0.26 velocity=5.4
- joint joint_left_aileron: limit lower=-0.3491 upper=0.3491 effort=5.0 velocity=5.4 -> lower=-0.3491 upper=0.3491 effort=0.26 velocity=5.4
- joint joint_right_aileron: limit lower=-0.3491 upper=0.3491 effort=5.0 velocity=5.4 -> lower=-0.3491 upper=0.3491 effort=0.26 velocity=5.4

File: genesis/assets/urdf/mydrone/mydrone_new.urdf (robot description, URDF)
Before this commit: robot drone_ea, 18 links, 17 joints
Links:
- link elevator: geometry collision box name=elevator_collision_0_box_0 size=0.013556761639149529 0.139941292987101 0.36000365939871676; visual mesh filename=package://meshes/elevator.stl name=elevator_visual_0_shape_0 scale=0.0007 0.0012 0.001
- link fuselage: geometry collision box name=fuselage_collision_0_box_0 size=0.10000000000000005 0.10476803794561983 0.7273891147638257; visual mesh filename=package://meshes/fuselage_only.stl name=fuselage_visual_0_shape_0 scale=0.00097 0.001 0.001
- link left_wing: geometry collision box name=left_wing_collision_0_box_0 size=0.01796222497680495 0.19998814444400242 0.7; visual mesh filename=package://meshes/wing0009.stl name=left_wing_visual_0_shape_0 scale=0.2 0.7 0.2
- link prop_frame_fuselage_0: geometry visual cylinder length=0.005 name=prop_frame_fuselage_0_visual_0_shape_0 radius=0.1
- link right_wing: geometry collision box name=right_wing_collision_0_box_0 size=0.01796222497680495 0.19998814444400242 0.7; visual mesh filename=package://meshes/wing0009.stl name=right_wing_visual_0_shape_0 scale=0.2 0.7 0.2
- link rudder: geometry collision box name=rudder_collision_0_box_0 size=0.01347209289684701 0.119323096637794 0.16357341166046455; visual mesh filename=package://meshes/rudder.stl name=rudder_visual_0_shape_0 scale=0.0008 0.001 0.001
Joints:
- joint elevator_pitch_joint: limit lower=-0.261799 upper=0.261799 effort=5 velocity=2 -> lower=-0.261799 upper=0.261799 effort=1.0 velocity=3.665191429
- joint fixed_joint_aero_frame_left_wing: origin xyz=0.034436664 -0.35 0 rpy=0 0 0 -> xyz=0.034436664 0.35 0 rpy=3.141592653589793 0 0
- joint fixed_joint_left_wing: origin xyz=-0.275 -0.05 -0.03 rpy=0 3.141592653589793 0 -> xyz=-0.275 -0.05 -0.03 rpy=0 0 3.141592653589793
- joint joint_0_twist_left_wing: axis 0 -1 0 -> 0 1 0; limit lower=-0.5235987756 upper=0.5235987756 effort=5 velocity=3.665191429 -> lower=-0.5235987756 upper=0.5235987756 effort=2.0 velocity=3.665191429
- joint joint_0_twist_right_wing: limit lower=-0.5235987756 upper=0.5235987756 effort=5 velocity=3.665191429 -> lower=-0.5235987756 upper=0.5235987756 effort=2.0 velocity=3.665191429
- joint rudder_yaw_joint: limit lower=-0.523599 upper=0.523599 effort=3 velocity=2.5 -> lower=-0.523599 upper=0.523599 effort=1.0 velocity=3.665191429
